File: project/kb1lqd_optical_comm/mic_preamp.sch (KiCad schematic (older format))
At the start: 17 parts, among them U2 AD8648

Commit message: Updated with all footprints
Parts:
- removed U2: AD8648, symbol kb1lqd_optical_comm:AD8648
- added U2: AD8646, Package_SO:TSSOP-8_3x3mm_P0.65mm, symbol kb1lqd_optical_comm:AD8646
- C21, C22: footprint (none) -> Capacitor_SMD:C_0603_1608Metric
- C23, C6: footprint (none) -> Capacitor_SMD:C_0805_2012Metric
- C4, C5, C7: footprint (none) -> Capacitor_SMD:C_1206_3216Metric
- R18, R19, R20, R21, R22, R23, R24: footprint (none) -> Resistor_SMD:R_0603_1608Metric
- R34: renamed from 100k1; value R_US -> 100k; footprint (none) -> Resistor_SMD:R_0805_2012Metric
- RV2: value 20k -> 50k; footprint (none) -> Connector_Molex:Molex_KK-254_AE-6410-04A_1x04_P2.54mm_Vertical
Connections:
- net +5V: now also U2.8 (V+)
- net AUDIO_OUTPUT: now also U2.7
- net GND: now also U2.4 (V-)
- net at C6.2, R20.1, R34.2: now also U2.3 (+)
- net at C6.1, C7.2, R34.1: now also U2.1
- net at R18.1, R19.2: now also U2.2 (-)
- net at C21.1, R21.1, R22.2: now also U2.6 (-)
- net at C22.2, R23.1, R24.2: now also U2.5 (+)
Other:
- note added: "Should be 20k, just using 50k panel mount I have on hand."
Changed lines of the file:
@@
 F 0 "R20" V 3795 3700 50  0000 C CNN
 F 1 "1k" V 3886 3700 50  0000 C CNN
-F 2 "" V 4040 3690 50  0001 C CNN
+F 2 "Resistor_SMD:R_0603_1608Metric" V 4040 3690 50  0001 C CNN
 F 3 "~" H 4000 3700 50  0001 C CNN
 	1    4000 3700
@@
 $EndComp
 $Comp
-L Device:R_US 100k1
+L Device:R_US R34
 U 1 1 5F64F8BA
 P 4850 3150
-F 0 "100k1" V 4645 3150 50  0000 C CNN
-F 1 "R_US" V 4736 3150 50  0000 C CNN
-F 2 "" V 4890 3140 50  0001 C CNN
+F 0 "R34" V 4645 3150 50  0000 C CNN
+F 1 "100k" V 4736 3150 50  0000 C CNN
+F 2 "Resistor_SMD:R_0805_2012Metric" V 4890 3140 50  0001 C CNN
 F 3 "~" H 4850 3150 50  0001 C CNN
 	1    4850 3150
 	0    1    1    0
-$EndComp
-$Comp
-L kb1lqd_optical_comm:AD8648 U2
-U 1 1 5F655125
-P 4100 3400
-F 0 "U2" H 4750 3433 50  0000 C CNN
-F 1 "AD8648" H 4750 3524 50  0000 C CNN
-F 2 "" H 4100 3400 50  0001 C CNN
-F 3 "" H 4100 3400 50  0001 C CNN
-	1    4100 3400
-	1    0    0    1
-$EndComp
-$Comp
-L kb1lqd_optical_comm:AD8648 U2
-U 2 1 5F6554DE
-P 6750 3500
-F 0 "U2" H 7400 3533 50  0000 C CNN
-F 1 "AD8648" H 7400 3624 50  0000 C CNN
-F 2 "" H 6750 3500 50  0001 C CNN
-F 3 "" H 6750 3500 50  0001 C CNN
-	2    6750 3500
-	1    0    0    1
-$EndComp
-$Comp
-L kb1lqd_optical_comm:AD8648 U2
-U 3 1 5F655A3E
-P 1600 6900
-F 0 "U2" H 2278 7301 50  0000 L CNN
-F 1 "AD8648" H 2278 7210 50  0000 L CNN
-F 2 "" H 1600 6900 50  0001 C CNN
-F 3 "" H 1600 6900 50  0001 C CNN
-	3    1600 6900
-	1    0    0    -1
 $EndComp
 $Comp
@@
 F 0 "R19" H 3432 4204 50  0000 R CNN
 F 1 "1k" H 3432 4295 50  0000 R CNN
-F 2 "" V 3540 4240 50  0001 C CNN
+F 2 "Resistor_SMD:R_0603_1608Metric" V 3540 4240 50  0001 C CNN
 F 3 "~" H 3500 4250 50  0001 C CNN
 	1    3500 4250
@@
 F 0 "R18" H 3432 3254 50  0000 R CNN
 F 1 "3.24k" H 3432 3345 50  0000 R CNN
-F 2 "" V 3540 3290 50  0001 C CNN
+F 2 "Resistor_SMD:R_0603_1608Metric" V 3540 3290 50  0001 C CNN
 F 3 "~" H 3500 3300 50  0001 C CNN
 	1    3500 3300
@@
 F 0 "C5" V 2748 3700 50  0000 C CNN
 F 1 "1u" V 2839 3700 50  0000 C CNN
-F 2 "" H 3038 3550 50  0001 C CNN
+F 2 "Capacitor_SMD:C_1206_3216Metric" H 3038 3550 50  0001 C CNN
 F 3 "~" H 3000 3700 50  0001 C CNN
 	1    3000 3700
@@
 F 0 "C7" V 5548 3800 50  0000 C CNN
 F 1 "1u" V 5639 3800 50  0000 C CNN
-F 2 "" H 5838 3650 50  0001 C CNN
+F 2 "Capacitor_SMD:C_1206_3216Metric" H 5838 3650 50  0001 C CNN
 F 3 "~" H 5800 3800 50  0001 C CNN
 	1    5800 3800
@@
 F 0 "R23" V 6445 3800 50  0000 C CNN
 F 1 "1k" V 6536 3800 50  0000 C CNN
-F 2 "" V 6690 3790 50  0001 C CNN
+F 2 "Resistor_SMD:R_0603_1608Metric" V 6690 3790 50  0001 C CNN
 F 3 "~" H 6650 3800 50  0001 C CNN
 	1    6650 3800
@@
 F 0 "R22" H 6082 4304 50  0000 R CNN
 F 1 "1k" H 6082 4395 50  0000 R CNN
-F 2 "" V 6190 4340 50  0001 C CNN
+F 2 "Resistor_SMD:R_0603_1608Metric" V 6190 4340 50  0001 C CNN
 F 3 "~" H 6150 4350 50  0001 C CNN
 	1    6150 4350
@@
 F 0 "R21" H 6082 3354 50  0000 R CNN
 F 1 "3.24k" H 6082 3445 50  0000 R CNN
-F 2 "" V 6190 3390 50  0001 C CNN
+F 2 "Resistor_SMD:R_0603_1608Metric" V 6190 3390 50  0001 C CNN
 F 3 "~" H 6150 3400 50  0001 C CNN
 	1    6150 3400
@@
 F 0 "R24" V 7245 3150 50  0000 C CNN
 F 1 "1k" V 7336 3150 50  0000 C CNN
-F 2 "" V 7490 3140 50  0001 C CNN
+F 2 "Resistor_SMD:R_0603_1608Metric" V 7490 3140 50  0001 C CNN
 F 3 "~" H 7450 3150 50  0001 C CNN
 	1    7450 3150
@@
 P 7950 3150
 F 0 "RV2" V 7745 3150 50  0000 C CNN
-F 1 "20k" V 7836 3150 50  0000 C CNN
-F 2 "" H 7950 3150 50  0001 C CNN
+F 1 "50k" V 7836 3150 50  0000 C CNN
+F 2 "Connector_Molex:Molex_KK-254_AE-6410-04A_1x04_P2.54mm_Vertical" H 7950 3150 50  0001 C CNN
 F 3 "~" H 7950 3150 50  0001 C CNN
 	1    7950 3150
@@
 F 0 "C4" H 1385 6604 50  0000 R CNN
 F 1 "1u" H 1385 6695 50  0000 R CNN
-F 2 "" H 1538 6500 50  0001 C CNN
+F 2 "Capacitor_SMD:C_1206_3216Metric" H 1538 6500 50  0001 C CNN
 F 3 "~" H 1500 6650 50  0001 C CNN
 	1    1500 6650
@@
 F 0 "C6" V 4598 2600 50  0000 C CNN
 F 1 "DNP" V 4689 2600 50  0000 C CNN
-F 2 "" H 4888 2450 50  0001 C CNN
+F 2 "Capacitor_SMD:C_0805_2012Metric" H 4888 2450 50  0001 C CNN
 F 3 "~" H 4850 2600 50  0001 C CNN
 	1    4850 2600
@@
 F 0 "C22" V 7398 2550 50  0000 C CNN
 F 1 "DNP" V 7489 2550 50  0000 C CNN
-F 2 "" H 7688 2400 50  0001 C CNN
+F 2 "Capacitor_SMD:C_0603_1608Metric" H 7688 2400 50  0001 C CNN
 F 3 "~" H 7650 2550 50  0001 C CNN
 	1    7650 2550
@@
 F 0 "C21" V 5548 4350 50  0000 C CNN
 F 1 "DNP" V 5639 4350 50  0000 C CNN
-F 2 "" H 5838 4200 50  0001 C CNN
+F 2 "Capacitor_SMD:C_0603_1608Metric" H 5838 4200 50  0001 C CNN
 F 3 "~" H 5800 4350 50  0001 C CNN
 	1    5800 4350
@@
 F 0 "C23" V 898 6650 50  0000 C CNN
 F 1 "100nF" V 989 6650 50  0000 C CNN
-F 2 "" H 1188 6500 50  0001 C CNN
+F 2 "Capacitor_SMD:C_0805_2012Metric" H 1188 6500 50  0001 C CNN
 F 3 "~" H 1150 6650 50  0001 C CNN
 	1    1150 6650
@@
 	1    0    0    -1
 $EndComp
+$Comp
+L kb1lqd_optical_comm:AD8646 U2
+U 1 1 5FD73C1E
+P 4100 4200
+F 0 "U2" H 4750 4967 50  0000 C CNN
+F 1 "AD8646" H 4750 4876 50  0000 C CNN
+F 2 "Package_SO:TSSOP-8_3x3mm_P0.65mm" H 4100 4200 50  0001 C CNN
+F 3 "" H 4100 4200 50  0001 C CNN
+	1    4100 4200
+	1    0    0    -1
+$EndComp
+$Comp
+L kb1lqd_optical_comm:AD8646 U2
+U 2 1 5FD745F0
+P 6750 4300
+F 0 "U2" H 7400 5067 50  0000 C CNN
+F 1 "AD8646" H 7400 4976 50  0000 C CNN
+F 2 "Package_SO:TSSOP-8_3x3mm_P0.65mm" H 6750 4300 50  0001 C CNN
+F 3 "" H 6750 4300 50  0001 C CNN
+	2    6750 4300
+	1    0    0    -1
+$EndComp
+$Comp
+L kb1lqd_optical_comm:AD8646 U2
+U 3 1 5FD7500F
+P 1600 6900
+F 0 "U2" H 2278 7301 50  0000 L CNN
+F 1 "AD8646" H 2278 7210 50  0000 L CNN
+F 2 "Package_SO:TSSOP-8_3x3mm_P0.65mm" H 1600 6900 50  0001 C CNN
+F 3 "" H 1600 6900 50  0001 C CNN
+	3    1600 6900
+	1    0    0    -1
+$EndComp
+Text Notes 8600 3000 0    50   ~ 0
+Should be 20k, just using 50k panel mount I have on hand.
 $EndSCHEMATC

Commit message: Updated u2 to soic 8
Parts:
- U2: footprint Package_SO:TSSOP-8_3x3mm_P0.65mm -> Package_SO:SOIC-8_3.9x4.9mm_P1.27mm
Changed lines of the file:
@@
 F 0 "U2" H 4750 4967 50  0000 C CNN
 F 1 "AD8646" H 4750 4876 50  0000 C CNN
-F 2 "Package_SO:TSSOP-8_3x3mm_P0.65mm" H 4100 4200 50  0001 C CNN
+F 2 "Package_SO:SOIC-8_3.9x4.9mm_P1.27mm" H 4100 4200 50  0001 C CNN
 F 3 "" H 4100 4200 50  0001 C CNN
 	1    4100 4200
@@
 F 0 "U2" H 7400 5067 50  0000 C CNN
 F 1 "AD8646" H 7400 4976 50  0000 C CNN
-F 2 "Package_SO:TSSOP-8_3x3mm_P0.65mm" H 6750 4300 50  0001 C CNN
+F 2 "Package_SO:SOIC-8_3.9x4.9mm_P1.27mm" H 6750 4300 50  0001 C CNN
 F 3 "" H 6750 4300 50  0001 C CNN
 	2    6750 4300
@@
 F 0 "U2" H 2278 7301 50  0000 L CNN
 F 1 "AD8646" H 2278 7210 50  0000 L CNN
-F 2 "Package_SO:TSSOP-8_3x3mm_P0.65mm" H 1600 6900 50  0001 C CNN
+F 2 "Package_SO:SOIC-8_3.9x4.9mm_P1.27mm" H 1600 6900 50  0001 C CNN
 F 3 "" H 1600 6900 50  0001 C CNN
 	3    1600 6900
